File: fpga.kicad_pcb (KiCad board)
At the start: 4 copper layers, 100 x 100 mm, 37 parts, among them IC1 XC3S200-4TQG144C, IC2 MIC5504-3.3YM5-TR, IC3 MIC5504-2.5YM5-T5, IC4 MIC5504-1.2YM5-TR, IC5 ATMEGA328P-PU, IC6 FT232RL-TUBE, J1 ICSP, J2 BANK 6/7, J3 55917-1410, J4 ZX62-B-5PA_33_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

Commit message: rotated USB connector
Parts:
- moved J4 65.5 mm to (156.3, 141.6), turned to 0 degrees
- moved C1 65.4 mm to (133.2, 136.8)
- moved C3 65.4 mm to (134.1, 125.3)
- moved C6 65.4 mm to (143.4, 125.0)
- moved IC3 65.4 mm to (129.4, 126.0)
- moved IC5 65.4 mm to (194.8, 126.6)
- moved J1 65.4 mm to (208.8, 138.0)
- moved J5 65.4 mm to (211.8, 75.8)
- moved R9 65.4 mm to (205.0, 113.3)
- moved S8 65.4 mm to (208.8, 122.2)
- moved C2 65.4 mm to (142.1, 136.5)
- moved C8 65.4 mm to (177.7, 140.0)
- moved IC4 65.4 mm to (141.5, 129.2)
- moved J3 65.4 mm to (129.3, 67.9)
- moved R1 65.4 mm to (129.4, 130.4)
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Routing:
- net D+: track 21.7 -> 14.3 mm
- net VBUS: track 76.5 -> 70.1 mm
- net D-: track 15.6 -> 18.8 mm
- net GND: track 61.1 -> 58.9 mm
